File: cdh-devkit.kicad_pcb (KiCad board)
At the start: 2 copper layers, 31 parts, among them J1 UART, J2 CAN, J3 SPI, J4 I2C, J5 SWD, J6 GPIO, J7 USB_B_Micro, U1 STM32L433RCT6, U2 AMS1117-3.3, U3 MX25V8035FM2I, Y1 16MHz

Commit message: version 0.1
Parts:
- removed the J1 at (112.4, 58.4)
- removed the J4 at (99.7, 52.7)
- removed J6: GPIO, Connector_PinHeader_2.54mm:PinHeader_1x05_P2.54mm_Vertical
- added D3: BLUE, LED_SMD:LED_0603_1608Metric, F.Cu at (37.8, 55.6)
- added H1: MountingHole_Pad, MountingHole:MountingHole_2.2mm_M2_Pad, F.Cu at (19.0, 19.0)
- added H2: MountingHole_Pad, MountingHole:MountingHole_2.2mm_M2_Pad, F.Cu at (56.0, 91.0)
- added H3: MountingHole_Pad, MountingHole:MountingHole_2.2mm_M2_Pad, F.Cu at (56.0, 19.0)
- added H4: MountingHole_Pad, MountingHole:MountingHole_2.2mm_M2_Pad, F.Cu at (19.0, 91.0)
- added R5: 1k5, Resistor_SMD:R_0402_1005Metric, F.Cu at (37.8, 53.1)
- added S1: PTS525SM15SMTR2LFS, Buttons:SW_PTS525SM15SMTR2LFS, F.Cu at (27.0, 19.0)
- added U4: DS1339U-33+T&R, MSOP:21-0036K, F.Cu at (42.7, 42.8)
- added Y2: 32.768K, Crystals:XTAL_NX3215SA-32.768K-STD-MUA-14, F.Cu at (37.5, 42.1)
- J2: value CAN -> Conn_01x15_Male; footprint Connector_PinHeader_2.54mm:PinHeader_1x04_P2.54mm_Vertical -> Connector_PinHeader_2.54mm:PinHeader_1x15_P2.54mm_Horizontal
- J3: value SPI -> Conn_01x09_Male; footprint Connector_PinHeader_2.54mm:PinHeader_1x05_P2.54mm_Vertical -> Connector_PinHeader_2.54mm:PinHeader_1x09_P2.54mm_Horizontal
- J4: renamed from J7; footprint Connector_USB:USB_Micro-B_Wuerth_629105150521 -> Connector_USB:USB_Micro-B_Molex-105017-0001
- moved J1 94.9 mm to (35.0, 89.2), turned to 90 degrees
- moved C13 69.2 mm to (28.2, 67.9), turned to 180 degrees
- moved R1 68.9 mm to (51.0, 16.5), turned to 90 degrees
- moved D2 65.2 mm to (51.0, 19.1), turned to -90 degrees
- moved C12 63.2 mm to (30.2, 66.2), turned to 90 degrees
- moved C11 56.2 mm to (23.2, 23.0), turned to 180 degrees
- moved J4 47.3 mm to (37.5, 17.7), turned to 180 degrees
- moved R3 42.7 mm to (44.9, 47.2)
- moved R4 42.1 mm to (42.6, 47.3)
- moved J3 41.8 mm to (57.3, 65.6), turned to 0 degrees
- moved C7 38.2 mm to (34.5, 71.5)
- moved C5 34.5 mm to (30.2, 60.0), turned to 90 degrees
- moved R2 34.3 mm to (46.0, 16.5), turned to 90 degrees
- moved D1 32.0 mm to (46.0, 19.1), turned to -90 degrees
- moved C3 31.7 mm to (44.8, 60.5)
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- renumbered C3 to C1, C8 to C10, C9 to C12, C10 to C13, C1 to C2, C4 to C3, C12 to C4, C2 to C6, C6 to C7, C13 to C8, C7 to C9, J5 to J1, R3 to R1, R4 to R3, R5 to R4, R1 to R6, U2 to U1, U1 to U2
Connections:
- net Net-(C12-Pad1) renamed /OSC_IN
- net Net-(C13-Pad1) renamed /OSC_OUT
- net Net-(D2-Pad2) renamed /USB_NOE
- C2 pad 2: Net-(C1-Pad2) -> GND
- C6 pad 2: Net-(C1-Pad2) -> GND
- J1 pad 1: SWDIO -> GND
- J1 pad 3: GND -> SWDIO
- J2 pad 1: GND -> +3.3V
- J2 pad 2: CAN_TX -> UART_TX
- J2 pad 3: CAN_RX -> UART_RX
- J2 pad 4: +3.3V -> GND
- J3 pad 2: SPI_SCK -> GND
- J3 pad 3: SPI_MISO -> GPIO_1
- J3 pad 4: SPI_MOSI -> GPIO_2
- J3 pad 5: GND -> GPIO_3
- J4 pad 6: unconnected-(J7-Pad6) -> GND
- R2 pad 2: Net-(C1-Pad2) -> GND
- U2 pad 33: unconnected-(U1-Pad33) -> GPIO_5
- U2 pad 34: unconnected-(U1-Pad34) -> GPIO_4
- U2 pad 35: unconnected-(U1-Pad35) -> GPIO_3
- U2 pad 36: unconnected-(U1-Pad36) -> GPIO_2
- U2 pad 37: unconnected-(U1-Pad37) -> GPIO_1
- U2 pad 55: GPIO_1 -> unconnected-(U2-Pad55)
- U2 pad 56: GPIO_2 -> unconnected-(U2-Pad56)
- U2 pad 57: GPIO_3 -> unconnected-(U2-Pad57)
- U2 pad 58: GPIO_4 -> /GPIO_LED
- U2 pad 59: GPIO_5 -> unconnected-(U2-Pad59)
Routing:
- net +3.3V: track 0.00 -> 258.5 mm, vias 0 -> 12
- net GND: track 0.00 -> 105.1 mm, vias 0 -> 26
- net D-: track 0.00 -> 59.3 mm, vias 0 -> 2
- net D+: track 0.00 -> 58.6 mm, vias 0 -> 2
- net /USB_NOE: track 0.00 -> 56.7 mm, vias 0 -> 2
- net UART_TX: track 0.00 -> 55.4 mm, vias 0 -> 2
- net Net-(C11-Pad1): track 0.00 -> 55.3 mm
- net UART_RX: track 0.00 -> 51.2 mm, vias 0 -> 2
- net CAN_TX: track 0.00 -> 47.1 mm
- net CAN_RX: track 0.00 -> 45.4 mm
- net I2C_SCL: track 0.00 -> 44.4 mm, vias 0 -> 2
- net I2C_SDA: track 0.00 -> 43.8 mm, vias 0 -> 2
- net SWCLK: track 0.00 -> 34.6 mm, vias 0 -> 1
- net SWDIO: track 0.00 -> 30.8 mm, vias 0 -> 1
- net QSPI_IO_1: track 0.00 -> 27.8 mm
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- added copper zone on F.Cu, net GND
- added copper zone on In1.Cu, net GND
- added copper zone on In2.Cu, net GND
Other:
- board outline added: 45 x 80 mm
- copper layers 2 -> 4
- board text added: "3.3V"
- board text added: "Addr: 0x68"
- board text added: "CAN_RX"
- board text added: "CAN_TX"
- board text added: "GND"
- board text added: "I2C_SCL"
- board text added: "I2C_SDA"
- board text added: "KRONOS DEV KIT"
- board text added: "PB12"
- board text added: "PB13"
- board text added: "PB14"
- board text added: "PB15"
- board text added: "PC6"
- board text added: "POWER"
- board text added: "Pin: PB6"
- board text added: "RESET"
- board text added: "SN: JLCJLCJLCJLC"
- board text added: "SPI_MISO"
- board text added: "SPI_MOSI"
- board text added: "SPI_SCK"
- board text added: "STM32L433RCT6"
- board text added: "SWCLK"
- board text added: "SWD"
- board text added: "SWDIO"
- board text added: "UART_RX"
- board text added: "UART_TX"
- board text added: "USB"
- board text added: "Version 1.0"
- board text removed: "CAN"
