File: cdh-devkit.kicad_sch (KiCad schematic)
At the start: 33 parts, among them J1 SWD, J2 Conn_01x15_Male, J3 Conn_01x09_Male, J4 USB_B_Micro, U1 AMS1117-3.3, U2 STM32L433RCT6, Y1 16MHz

Commit message: started rerouting
Parts:
- R3, R4: value 1k5 -> 10k
Changed lines of the file:
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@@
     (stroke (width 0) (type default) (color 0 0 0 0))
   )
-  (wire (pts (xy 35.56 189.23) (xy 35.56 191.77))
+  (wire (pts (xy 35.56 189.23) (xy 35.56 194.31))
     (stroke (width 0) (type default) (color 0 0 0 0))
   )
@@
     (stroke (width 0) (type default) (color 0 0 0 0))
   )
-  (wire (pts (xy 38.1 189.23) (xy 38.1 191.77))
+  (wire (pts (xy 38.1 189.23) (xy 38.1 194.31))
     (stroke (width 0) (type default) (color 0 0 0 0))
   )
@@
     )
   )
-  (global_label "D+" (shape input) (at 38.1 191.77 270) (fields_autoplaced)
+  (global_label "D+" (shape input) (at 38.1 194.31 270) (fields_autoplaced)
     (effects (font (size 1 1)) (justify right))
-    (property "Intersheet References" "${INTERSHEET_REFS}" (id 0) (at 38.0375 195.9081 90)
+    (property "Intersheet References" "${INTERSHEET_REFS}" (id 0) (at 38.0375 198.4481 90)
       (effects (font (size 1 1)) (justify left) hide)
     )
@@
     )
   )
-  (global_label "D-" (shape input) (at 35.56 191.77 270) (fields_autoplaced)
+  (global_label "D-" (shape input) (at 35.56 194.31 270) (fields_autoplaced)
     (effects (font (size 1 1)) (justify right))
-    (property "Intersheet References" "${INTERSHEET_REFS}" (id 0) (at 35.4975 195.9081 90)
+    (property "Intersheet References" "${INTERSHEET_REFS}" (id 0) (at 35.4975 198.4481 90)
       (effects (font (size 1 1)) (justify left) hide)
     )
@@
       (effects (font (size 1.27 1.27)) (justify left))
     )
-    (property "Value" "1k5" (id 1) (at 222.25 138.43 0)
+    (property "Value" "10k" (id 1) (at 222.25 138.43 0)
       (effects (font (size 1.27 1.27)) (justify left))
     )
@@
       (effects (font (size 1.27 1.27)) (justify left))
     )
-    (property "Value" "1k5" (id 1) (at 213.36 138.43 0)
+    (property "Value" "10k" (id 1) (at 213.36 138.43 0)
       (effects (font (size 1.27 1.27)) (justify left))
     )
@@
     )
     (path "/84a221cf-789d-4597-949e-8d2a5b3d9871"
-      (reference "R3") (unit 1) (value "1k5") (footprint "Resistor_SMD:R_0402_1005Metric")
+      (reference "R3") (unit 1) (value "10k") (footprint "Resistor_SMD:R_0402_1005Metric")
     )
     (path "/1a67957e-2f14-46bc-b565-cecca45e3d5e"
-      (reference "R4") (unit 1) (value "1k5") (footprint "Resistor_SMD:R_0402_1005Metric")
+      (reference "R4") (unit 1) (value "10k") (footprint "Resistor_SMD:R_0402_1005Metric")
     )
     (path "/54a4a5a3-f0a3-4336-90f2-3de63094bbc0"

Commit message: finished second revision
Parts:
- removed J1: SWD, Connector_PinHeader_2.54mm:PinHeader_1x03_P2.54mm_Vertical, symbol Connector:Conn_01x03_Male
- removed J2: Conn_01x15_Male, Connector_PinHeader_2.54mm:PinHeader_1x15_P2.54mm_Horizontal, symbol Connector:Conn_01x15_Male
- removed J3: Conn_01x09_Male, Connector_PinHeader_2.54mm:PinHeader_1x09_P2.54mm_Horizontal, symbol Connector:Conn_01x09_Male
- added J1, J2, J3: Conn_01x08_Male, Connector_PinHeader_2.54mm:PinHeader_1x08_P2.54mm_Vertical, symbol Connector:Conn_01x08_Male
- added R10, R11, R12, R13, R14, R15, R16, R17, R18, R3, R4, R5, R6, R7, R8, R9: 1K, Resistor_SMD:R_0402_1005Metric, symbol Device:R
- renumbered R3 to R19, R4 to R20, R5 to R21
Connections:
- net +3.3V: now also J1.1 (Pin_1), J1.8 (Pin_8), J2.1 (Pin_1), J2.8 (Pin_8), J3.1 (Pin_1), J3.8 (Pin_8)
- net CAN_RX: now also J1.6 (Pin_6), R15.1, R15.2
- net CAN_TX: now also J1.5 (Pin_5), R16.1, R16.2
- net GND: now also J1.4 (Pin_4), J1.7 (Pin_7), J2.4 (Pin_4), J3.7 (Pin_7)
- net GPIO_1: now also J3.2 (Pin_2), R6.1, R6.2
- net GPIO_2: now also J3.3 (Pin_3), R10.1, R10.2
- net GPIO_3: now also J3.4 (Pin_4), R9.1, R9.2
- net GPIO_4: now also J3.5 (Pin_5), R7.1, R7.2
- net GPIO_5: now also J3.6 (Pin_6), R8.1, R8.2
- net I2C_SCL: now also J2.2 (Pin_2), R17.1, R17.2
- net I2C_SDA: now also J2.3 (Pin_3), R18.1, R18.2
- net SPI_MISO: now also J2.6 (Pin_6), R4.1, R4.2
- net SPI_MOSI: now also J2.5 (Pin_5), R5.1, R5.2
- net SPI_SCK: now also J2.7 (Pin_7), R3.1, R3.2
- net SWCLK: now also R14.1, R14.2
- net SWDIO: now also R13.1, R13.2
- net UART_RX: now also J1.3 (Pin_3), R12.1, R12.2
- net UART_TX: now also J1.2 (Pin_2), R11.1, R11.2
Other:
- moved on the sheet: R19, R20, R21
