File: untitled.kicad_sch (KiCad schematic)
At the start: 4 parts, among them U3 MX25V8035FM2I

Commit message: version 0.1
Parts:
- Y2: renamed from Y?; footprint XTAL_NX3215SA-32.768K-STD-MUA-14 -> Crystals:XTAL_NX3215SA-32.768K-STD-MUA-14
- gave numbers to parts that had none: 1
- renumbered R1 to R6
Connections:
- net GND: now also U4.3 (VBACKUP)
- no-connect marks 2 -> 1
Other:
- moved on the sheet: R6, U4, Y2

Commit message: finished second revision
Parts:
- added D4: PESD2USB3UV-TR, SOT95P230X110-3N, symbol TVS:PESD2USB3UV-TR
- added J5: SWD, Connector_PinHeader_2.54mm:PinHeader_1x03_P2.54mm_Vertical, symbol Connector:Conn_01x03_Male
- added U4, U5, U6: DT1240A-08LP3810-7, TVS:TVS_824014883, symbol TVS:DT1240A-08LP3810-7
- renumbered R6 to R22, U4 to U7
Connections:
- net GND: now also D4.3 (COMMON_ANODE), J5.1 (Pin_1), U4.3 (GND), U5.3 (GND), U6.3 (GND)
- net I2C_SCL: now also U5.1 (LINE-1)
- net I2C_SDA: now also U5.2 (LINE-3)
- new net CAN_RX: U4.5 (LINE-8)
- new net CAN_TX: U4.4 (LINE-6)
- new net D+: D4.2 (CATHODE_(DIODE_2))
- new net D-: D4.1 (CATHODE_(DIODE_1))
- new net GPIO_1: U6.1 (LINE-1)
- new net GPIO_2: U6.2 (LINE-3)
- new net GPIO_3: U6.4 (LINE-6)
- new net GPIO_4: U6.5 (LINE-8)
- new net GPIO_5: U6.9 (LINE-2)
- new net SPI_MISO: U5.8 (LINE-4)
- new net SPI_MOSI: U5.9 (LINE-2)
- new net SPI_SCK: U5.7 (LINE-5)
- new net SWCLK: J5.2 (Pin_2), U5.6 (LINE-7)
- new net SWDIO: J5.3 (Pin_3), U5.5 (LINE-8)
- new net UART_RX: U4.2 (LINE-3)
- new net UART_TX: U4.1 (LINE-1)
- no-connect marks 1 -> 9
Other:
- note added: "Debug (SWD)"
- note added: "ESD Protection"
